File: OTMAKSTM32H05_64PIN/BLE_MOBILE.kicad_sch (KiCad schematic)
At the start: 41 parts, among them J17 PROG, SW2 BOOT_, SW2 EN, U1 QFN48, Y1 32.7680 KHz 12.5 pF, Y2 32.0000 MHz 8pF

Commit message: revision skematik
Connections:
- net UART_TXD_STM renamed UART_TXD_BLE
Changed lines of the file:
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@@
 	(generator_version "8.0")
 	(paper "A3")
+	(title_block
+		(date "2024-12-06")
+	)
 	(junction
 		(at 232.41 97.155)
@@
 	(wire
 		(pts
-			(xy 280.67 128.27) (xy 280.67 135.89)
+			(xy 280.67 128.27) (xy 280.67 140.97)
 		)
 		(stroke
@@
 	(wire
 		(pts
-			(xy 266.7 135.89) (xy 280.67 135.89)
+			(xy 266.7 140.97) (xy 280.67 140.97)
 		)
 		(stroke
@@
 	(wire
 		(pts
-			(xy 266.7 128.27) (xy 266.7 135.89)
+			(xy 266.7 128.27) (xy 266.7 140.97)
 		)
 		(stroke
@@
 		)
 	)
-	(hierarchical_label "UART_RXD_STM"
+	(hierarchical_label "UART_RXD_BLE"
 		(shape input)
 		(at 166.0906 167.767 0)
@@
 		)
 	)
-	(hierarchical_label "UART_TXD_STM"
+	(hierarchical_label "UART_TXD_BLE"
 		(shape input)
 		(at 288.29 128.27 270)
@@
 		(dnp no)
 		(property "Reference" "C1"
-			(at 100.8126 133.8834 0)
+			(at 104.14 132.588 90)
 			(effects
 				(font
@@
 		)
 		(property "Value" "100nF"
-			(at 100.5078 137.9982 90)
+			(at 100.076 137.16 90)
 			(effects
 				(font

Commit message: next revisi 241206 1656
Connections:
- net UART_TXD_BLE renamed UART_TXD_STM
Changed lines of the file:
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@@
 		)
 	)
-	(hierarchical_label "UART_RXD_BLE"
+	(hierarchical_label "UART_RXD_STM"
 		(shape input)
 		(at 166.0906 167.767 0)
@@
 		)
 	)
-	(hierarchical_label "UART_TXD_BLE"
+	(hierarchical_label "UART_TXD_STM"
 		(shape input)
 		(at 288.29 128.27 270)
@@
 			(project "OTMAK"
 				(path "/ba4d3907-32eb-4339-b757-c61b0e168373/be1b7685-73c2-4664-a1d8-321c44fee7dd"
-					(reference "C28")
+					(reference "C27")
 					(unit 1)
 				)

Commit message: full version
Parts:
- removed R5: 100K, Resistor_SMD:R_0603_1608Metric, symbol Device:R
- removed R6: 100R, Resistor_SMD:R_0603_1608Metric, symbol Device:R
- added R18: 100R, Resistor_SMD:R_0603_1608Metric, symbol Device:R
- added R21: 100K, Resistor_SMD:R_0603_1608Metric, symbol Device:R
- added TP13, TP14, TP15: ~, TestPoint:TestPoint_Loop_D2.50mm_Drill1.0mm, symbol Connector:TestPoint
- SW2: footprint TS-1187A-B-A-B:SW_TS-1187A-B-A-B -> Push Button:KEY-SMD_4P-L4.2-W3.2-P2.20-LS4.6
Connections:
- net 3V3: now also R18.1
- net BOOTA: now also SW2.1, SW2.2, R21.1; no longer SW2.C (A), SW2.D (3)
- net GNDREF: now also R21.2
- net RSTN: now also SW2.1, SW2.2; no longer SW2.A (1), SW2.B (2)
- net at U1.13 (PA0): now also TP13.1
- net at U1.42 (PB10): now also TP14.1
- net at U1.8 (PA12): now also TP15.1
- new net: R18.2, SW2.3, SW2.4
- new net: R2.1, SW2.3, SW2.4
- no-connect marks 22 -> 16
Other:
- moved on the sheet: D2, R8, SW2
