File: OTMAKSTM32H05_64PIN/OTMAK.kicad_pcb (KiCad board)
At the start: 2 copper layers, 160 x 114.3 mm, 222 parts, among them J1 TYPE-C-31-M-12, J10 TX_DEBUG, J11 Conn_01x01, J12 Conn_01x08, J13 Conn_01x08, J15 Conn_01x08, J16 Conn_01x08, J17 PROG, J18 IR Interrupt, J19 Conn_01x08, J2 TYPE-C-31-M-12, J20 MOTOR_A/MOTOR_B, J21 24V INPUT, J3 TYPE-C-31-M-12, J4 TYPE-C-31-M-12, J5 TYPE-C-31-M-12, J6 RJ45, J7 STLink, J8 RJ45, J9 RX_DEBUG, Q1 BSS138, SW1 EN, SW3 EN, SW4 BOOT_, U11 LM393, U12 CC6900SO-20A, U15 LM1117-3.3, U2 W25Q128JVSIQ, U6 QFN48, Y1 25.00Mhz, 50PPM, Y2 32.768 kHz, Y3 32.7680 KHz 12.5 pF, Y4 32.0000 MHz 8pF

Commit message: next revisi 241206 1656
Parts:
- removed the C20 at (154.0, 62.0)
- removed the C22 at (192.5, 46.1)
- removed the C23 at (154.0, 63.9)
- removed C54, C55: 10nF, Capacitor_SMD:C_0603_1608Metric
- removed C57, C58: 100nF, Capacitor_SMD:C_1206_3216Metric
- removed C60, C61: 470uF/1000uF, Capacitor_SMD:CP_Elec_10x10.5
- removed C79, C82: 1uF, Capacitor_SMD:C_0805_2012Metric
- removed C81, C84: 100nF, Capacitor_SMD:C_0805_2012Metric
- removed FB2: 600 @ 100mhz, Inductor_SMD:L_0603_1608Metric
- removed J19: Conn_01x08, Terminal_8_pin:TerminalBlock_8_pin
- removed J20: MOTOR_A/MOTOR_B, Terminal_4_pin:TerminalBlock_4_pin
- removed J4: TYPE-C-31-M-12, TYPE-C-31-M-12:HRO_TYPE-C-31-M-12
- removed R33: 10K, Capacitor_SMD:C_0603_1608Metric
- removed R34: 0.51K, Resistor_SMD:R_0603_1608Metric
- removed R35: 0.51K, Resistor_SMD:R_0805_2012Metric
- removed R38, R39: 10K, Resistor_SMD:R_0603_1608Metric
- removed R41, R43: 47K, Resistor_SMD:R_0603_1608Metric
- removed R42, R44: 0R, Resistor_SMD:R_0805_2012Metric
- removed U15: LM1117-3.3, Package_TO_SOT_SMD:SOT-223-3_TabPin2
- removed U8: ~, Package_TO_SOT_SMD:TO-263-7_TabPin8
- added C27: 1nF, Capacitor_SMD:C_0603_1608Metric, F.Cu at (-63.6, 46.8)
- added C6: 2.2uF, Capacitor_SMD:C_0402_1005Metric, F.Cu at (-53.0, 72.9)
- added C7: 2.2uF, Capacitor_SMD:C_0402_1005Metric, F.Cu at (-53.0, 74.9)
- added C88: 4.7nF, Capacitor_SMD:C_0805_2012Metric, F.Cu at (-40.8, 65.4)
- added J6: MOTOR_A/MOTOR_B, TerminalBlock:TerminalBlock_bornier-6_P5.08mm, F.Cu at (2.89, 35.0)
- added J8: ROTARY, TerminalBlock:TerminalBlock_bornier-3_P5.08mm, F.Cu at (2.86, 44.1)
- added R17: 1K, Resistor_SMD:R_0603_1608Metric, F.Cu at (-63.6, 59.3)
- added R19: 10K, Capacitor_SMD:C_0603_1608Metric, F.Cu at (-59.6, 46.8)
- added R6: 52.3K, Resistor_SMD:R_0603_1608Metric, F.Cu at (-63.6, 54.3)
- added R8: 5k1, Resistor_SMD:R_0402_1005Metric, F.Cu at (-54.4, 83.4)
- added TP8: ~, TestPoint:TestPoint_Loop_D2.50mm_Drill1.0mm, F.Cu at (-58.2, 84.7)
- added U16: USBLC6-2SC6, Package_TO_SOT_SMD:SOT-23-6, F.Cu at (-63.1, 84.8)
- C12: value 10uF -> 1uF
- C13: renamed from C14; value 10uF -> 1uF
- C14: renamed from C15; value 10uF -> 1uF
- C15: renamed from C16; value 10uF -> 1uF
- C2, C3: value 6.8pF -> 24pF
- C48: value 1nF -> 100nF
- C49: value 1nF -> 1uF; footprint Capacitor_SMD:C_0805_2012Metric -> Capacitor_SMD:C_0603_1608Metric
- C51: footprint Capacitor_SMD:C_0603_1608Metric -> Capacitor_SMD:C_1206_3216Metric
- C52: value 100nF -> 470uF/1000uF; footprint Capacitor_SMD:C_0805_2012Metric -> Capacitor_SMD:CP_Elec_10x10.5
- C56, C65: value 10nF -> 1uF
- C75: value 22uF -> 4.7uF
- C76: value 10uF -> 4.7nF
- J5: footprint TYPE-C-31-M-12:HRO_TYPE-C-31-M-12 -> USB_Type_C:HRO_TYPE-C-31-M-12
- R14: value 5k1 -> 30.1K; footprint Resistor_SMD:R_0402_1005Metric -> Resistor_SMD:R_0603_1608Metric
- R26: value 1K -> 10K; footprint Resistor_SMD:R_0603_1608Metric -> Capacitor_SMD:C_0603_1608Metric
- R27: value 1K -> 0.51K; footprint Resistor_SMD:R_0805_2012Metric -> Resistor_SMD:R_0603_1608Metric
- R29: value 10K -> 3.9K; footprint Capacitor_SMD:C_0603_1608Metric -> Resistor_SMD:R_0603_1608Metric
- R30: value 10K -> 33K; footprint Capacitor_SMD:C_0603_1608Metric -> Resistor_SMD:R_0603_1608Metric
- R32: value 10K -> 0R; footprint Capacitor_SMD:C_0603_1608Metric -> Resistor_SMD:R_0805_2012Metric
- R40, R49: value 10K -> 3.9K
- R45, R47: value 47K -> 33K
- Y1: value 25.00Mhz, 50PPM -> 24MHz, 6pF
- moved TP7 212.8 mm to (-63.3, 62.9)
- moved J5 205.2 mm to (-60.0, 79.0), turned to 0 degrees
- moved R14 203.4 mm to (-63.6, 56.8), turned to 0 degrees
- moved R12 200.8 mm to (-54.4, 85.4), turned to 0 degrees
- moved C48 185.2 mm to (-63.6, 49.3)
- moved C51 182.2 mm to (-62.8, 66.9)
- moved C75 170.7 mm to (-40.8, 59.4)
- moved C76 170.7 mm to (-40.8, 62.4)
- moved R29 162.9 mm to (-59.6, 54.3)
- moved R26 161.7 mm to (-59.6, 49.3)
- moved C49 153.2 mm to (-63.6, 51.8)
- moved R27 145.5 mm to (-59.6, 51.8)
- moved R32 143.3 mm to (-40.8, 68.4)
- moved R30 141.5 mm to (-59.6, 56.8)
- moved C52 138.4 mm to (-50.2, 63.9)
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- renumbered C18 to C16, C19 to C17, C21 to C18, C17 to C19, C25 to C20, C27 to C21, C26 to C22, C24 to C23, C13 to C24, C6 to C25, C7 to C26, J8 to Remote1, J6 to SC1
Connections:
- net TM1_CH4 renamed ADC2_INP13
- C16 pad 2: VREF+ -> VDDA
- C17 pad 2: VREF+ -> VDDA
- C48 pad 1: Net-(U7-IS) -> Net-(U7-SR)
- C49 pad 1: Net-(U8-IS) -> Net-(C49-Pad1)
- C51 pad 1: Net-(U7-SR) -> IN-24V
- C52 pad 1: Net-(U8-SR) -> IN-24V
- C56 pad 2: Net-(C56-Pad2) -> VSS
- C65 pad 2: Net-(C65-Pad2) -> VSS
- C76 pad 1: 5V -> 3V3
- C76 pad 2: VSS -> Net-(U4-NR/FB)
- COM-TO-STM1 pad 3: USART3_TX_STM -> USART3_RX_STM
- COM-TO-STM1 pad 6: USART3_TX_STM -> USART3_RX_STM
- FB1 pad 2: VREF+ -> VDDA
- J1 pad A6: I2C_SDA -> I2C1_SDA
- J1 pad A7: I2C_SCL -> I2C1_SCL
- J1 pad B6: I2C_SDA -> I2C1_SDA
- J1 pad B7: I2C_SCL -> I2C1_SCL
- J17 pad 3: USART3_RX_STM -> USART3_TX_STM
- J2 pad A6: UART4_RX -> UART4_RX_LIDAR
- J2 pad A7: UART4_TX -> UART4_TX_LIDAR
- J2 pad B6: UART4_TX -> UART4_TX_LIDAR
- J2 pad B7: UART4_RX -> UART4_RX_LIDAR
- J5 pad A4B9: 5V -> Net-(D2-A)
- J5 pad A6: LPUART1_RX -> C_D+
- J5 pad A7: LPUART1_TX -> C_D-
- J5 pad B4A9: 5V -> Net-(D2-A)
- J5 pad B6: LPUART1_RX -> C_D+
- J5 pad B7: LPUART1_TX -> C_D-
- J7 pad 13: USART1_RX -> USART1_RX_ST-LINK
- J7 pad 14: USART1_TX -> USART1_TX_ST-LINK
- Q1 pad 1: BUZZER -> TIM2_CH2_BUZZER
- R11 pad 2: BUZZER -> TIM2_CH2_BUZZER
- R12 pad 1: VSS -> Net-(J5-CC2)
- R12 pad 2: Net-(J5-CC1) -> VSS
- R14 pad 1: Net-(J5-CC2) -> Net-(U4-NR/FB)
- R15 pad 1: RESETPIN -> SPI1_RESET
- R16 pad 1: LED1 -> LD1
- R18 pad 1: RESETPIN -> SPI1_RESET
- R26 pad 1: VSS -> TIM8_CH4
- R26 pad 2: Net-(U7-IS) -> Net-(U7-INH)
- R27 pad 2: Net-(U8-IS) -> Net-(U7-SR)
- R29 pad 1: IN4 -> Net-(C49-Pad1)
- R29 pad 2: Net-(U7-IN) -> VSS
- R30 pad 1: IN4 -> ROTARY_DC_OUT
- R30 pad 2: Net-(U8-IN) -> Net-(C49-Pad1)
- R31 pad 1: IN1 -> TIM3_CH1
- R32 pad 2: Net-(U7-INH) -> Net-(C49-Pad1)
- R36 pad 1: TM1_CH1 -> TIM8_CH3
- R40 pad 2: Net-(C56-Pad2) -> VSS
- R46 pad 1: ADC1_IN3 -> ADC2_INP11
- R48 pad 1: ADC1_IN2 -> ADC2_INP12
- R49 pad 2: Net-(C65-Pad2) -> VSS
- R55 pad 2: TM1_CH3 -> TIM3_CH4
- R56 pad 2: IN3 -> TIM3_CH2
- TP2 pad 1: PB9 -> PD2
- TP3 pad 1: SPI3_CS -> SPI2_CS
- TP4 pad 1: SPI3_CLK -> SPI2_CLK
- TP5 pad 1: SPI3_MOSI -> SPI2_MOSI
- TP6 pad 1: SPI3_MISO -> SPI2_MISO
- U1 pad 10: TM1_CH3 -> ADC1_INP12
- U1 pad 12: ADC1_IN1 -> VSSA
- U1 pad 13: ADC1_IN2 -> VDDA
- U1 pad 14: ADC1_IN3 -> ADC1_INP0
- U1 pad 15: VSS -> TIM2_CH2_BUZZER
- U1 pad 16: 3V3 -> USART2_TX_PSU
- U1 pad 17: ADC1_IN4 -> USART2_RX_PSU
- U1 pad 18: SPI1_NSS -> VSS
- U1 pad 19: SPI1_CLK -> 3V3
- U1 pad 2: unconnected-(U1-PC13-Pad2) -> PC13
- U1 pad 20: SPI1_MISO -> SPI1_CS1
- U1 pad 21: SPI1_MOSI -> SPI1_SCK
- U1 pad 22: INPUT_Foot_LOCK -> SPI1_MISO
- U1 pad 23: IN1 -> SPI1_MOSI
- U1 pad 24: unconnected-(U1-PB0-Pad24) -> USART3_RX_BLE
- U1 pad 25: IN3 -> SPI1_RESET
- U1 pad 26: IN4 -> SPI2_CS
- U1 pad 27: VSSA -> TIM3_CH4
- U1 pad 28: VREF+ -> SPI1_CS2
- U1 pad 29: VDDA -> USART3_TX_BLE
- U1 pad 30: USART3_TX_STM -> VCAP1
- U1 pad 33: USART3_RX_STM -> TIM8_CH3
- U1 pad 34: SPI2_NSS -> SPI2_CLK
- U1 pad 35: LED1 -> SPI2_MISO
- U1 pad 36: ADC1_IN5 -> SPI2_MOSI
- U1 pad 37: RESETPIN -> TIM3_CH1
- U1 pad 38: I2C_SCL -> TIM3_CH2
- U1 pad 39: I2C_SDA -> TIM3_CH3
- U1 pad 40: I2C3_SCL -> TIM8_CH4
- U1 pad 41: I2C3_SDA -> I2C3_SCL
- U1 pad 42: TM1_CH1 -> USART1_TX_ST-LINK
- U1 pad 43: USART1_TX -> USART1_RX_ST-LINK
- U1 pad 44: USART1_RX -> USB-DM
- U1 pad 45: unconnected-(U1-PA11-Pad45) -> USB-DP
- U1 pad 46: unconnected-(U1-PA12-Pad46) -> SWDIO
- U1 pad 49: SWDIO -> SWCLK
- U1 pad 50: SWCLK -> INPUT_Foot_LOCK
- U1 pad 51: SPI3_CS -> UART4_TX_LIDAR
- U1 pad 52: UART4_TX -> UART4_RX_LIDAR
- U1 pad 53: UART4_RX -> LD1
- U1 pad 54: UART5_TX_SC -> PD2
- U1 pad 55: UART5_RX_SC -> Rotary_GPIO_Read
- U1 pad 56: SPI3_CLK -> I2C3_SDA
- U1 pad 57: SPI3_MISO -> UART5_RX_SC
- U1 pad 58: SPI3_MOSI -> UART5_TX_SC
- U1 pad 59: BUZZER -> I2C1_SDA
- U1 pad 60: Rotary_GPIO_Read -> BOOT
- U1 pad 61: BOOT -> I2C1_SCL
- U1 pad 62: PB9 -> VCAP2
- U1 pad 8: LPUART1_RX -> PC0
- U1 pad 9: LPUART1_TX -> ADC2_INP11
- U12 pad 7: ADC1_IN1 -> ADC1_INP0
- U2 pad 1: SPI3_CS -> SPI2_CS
- U2 pad 2: SPI3_MISO -> SPI2_MISO
- U2 pad 5: SPI3_MOSI -> SPI2_MOSI
- U2 pad 6: SPI3_CLK -> SPI2_CLK
- U3 pad 17: SPI1_NSS -> SPI1_CS1
- U5 pad 17: SPI2_NSS -> SPI1_CS2
- U6 pad 11: USART3_RX_STM -> USART3_TX_STM

Commit message: full version
Parts:
- removed C21: 0.1uF, Capacitor_SMD:C_0805_2012Metric
- removed D9: BZV55B5V1, Diode_SMD:D_MiniMELF
- removed J6: MOTOR_A/MOTOR_B, TerminalBlock:TerminalBlock_bornier-6_P5.08mm
- removed R22: 100R, Resistor_SMD:R_0603_1608Metric
- added C54: 4.7uF, Capacitor_SMD:C_0805_2012Metric, F.Cu at (107.0, 100.3)
- added C55: 4.7nF, Capacitor_SMD:C_0805_2012Metric, F.Cu at (107.3, 106.8)
- added C57: 4.7nF, Capacitor_SMD:C_0805_2012Metric, F.Cu at (107.3, 108.9)
- added C58: 100nF, Capacitor_SMD:C_0402_1005Metric, F.Cu at (162.3, 66.3)
- added C60: 22uF, Capacitor_SMD:C_0805_2012Metric, F.Cu at (157.3, 46.5)
- added D2: D, Diode_SMD:D_SOD-123, F.Cu at (203.2, 53.2)
- added G***: LOGO, MAK:mak, F.Cu at (160.1, 100.9)
- added J14: TYPE-C-31-M-12, USB_Type_C:HRO_TYPE-C-31-M-12, F.Cu at (151.2, 38.9)
- added J19: Conn_01x02, TerminalBlock_2_pin:TerminalBlock_2_Pin, F.Cu at (93.5, 41.0)
- added J20: Conn_01x02, TerminalBlock_2_pin:TerminalBlock_2_Pin, F.Cu at (77.5, 41.1)
- added J22: Conn_01x02, TerminalBlock_2_pin:TerminalBlock_2_Pin, F.Cu at (106.4, 41.0)
- added J4: TYPE-C-31-M-12, USB_Type_C:HRO_TYPE-C-31-M-12, F.Cu at (138.2, 39.0)
- added R33: 52.3K, Resistor_SMD:R_0603_1608Metric, F.Cu at (110.1, 103.9)
- added R34: 30.1K, Resistor_SMD:R_0603_1608Metric, F.Cu at (104.7, 107.3)
- added R35: 5k1, Resistor_SMD:R_0402_1005Metric, F.Cu at (152.9, 47.0)
- added R38: 5k1, Resistor_SMD:R_0402_1005Metric, F.Cu at (149.1, 47.0)
- added TP10: ~, TestPoint:TestPoint_Loop_D2.50mm_Drill1.0mm, F.Cu at (153.7, 57.0)
- added TP11: ~, TestPoint:TestPoint_Loop_D2.50mm_Drill1.0mm, F.Cu at (114.7, 102.5)
- added TP12: ~, TestPoint:TestPoint_Loop_D2.50mm_Drill1.0mm, F.Cu at (100.4, 124.9)
- added TP13: ~, TestPoint:TestPoint_Loop_D2.50mm_Drill1.0mm, F.Cu at (214.4, 81.7)
- added TP14: ~, TestPoint:TestPoint_Loop_D2.50mm_Drill1.0mm, F.Cu at (187.1, 75.4)
- added TP15: ~, TestPoint:TestPoint_Loop_D2.50mm_Drill1.0mm, F.Cu at (202.0, 89.4)
- added TP9: ~, TestPoint:TestPoint_Loop_D2.50mm_Drill1.0mm, F.Cu at (112.3, 98.2)
- added U4: TPS73601DBVR, Package_TO_SOT_SMD:TSOT-23-5, F.Cu at (108.1, 114.9)
- added U8: TPS73601DBVR, Package_TO_SOT_SMD:TSOT-23-5, F.Cu at (107.0, 103.7)
- added ZD1: BZX55C5V1, BZX55C5V1:DO-35_BD2.0-L4.0-P8.00-D0.5-FD, F.Cu at (112.2, 93.6)
- C67, C68: footprint Capacitor_SMD:C_0805_2012Metric -> Capacitor_SMD:C_0603_1608Metric
- D8: footprint PDS4150:PDS4150 -> PDS4150-13:POWERDI-5_L5.4-W4.0-LS6.5-RD
- F1: footprint FuseSA72SB0:RES-SMD_SA72SB0 -> fuseSA72SB0:RES-SMD_SA72SB0
- J1, J2, J3: footprint TYPE-C-31-M-12:HRO_TYPE-C-31-M-12 -> USB_Type_C:HRO_TYPE-C-31-M-12
- J12, J13, J15, J16: footprint Terminal_8_pin:TerminalBlock_8_pin -> TerminalBlock_8_pin:TerminalBlock_8_pin
- J18: footprint Terminal_3_pin:TerminalBlock_3_Pin -> Terminal_3_Pin:TerminalBlock_3_Pin
- J8: footprint TerminalBlock:TerminalBlock_bornier-3_P5.08mm -> TerminalBlock_3_pin:TerminalBlock_3_Pin
- R18: footprint Resistor_SMD:R_0402_1005Metric -> Resistor_SMD:R_0603_1608Metric
- R58: footprint Resistor_SMD:R_0805_2012Metric -> Resistor_SMD:R_0603_1608Metric
- SW1, SW3, SW4: footprint TS-1187A-B-A-B:SW_TS-1187A-B-A-B -> Push Button:KEY-SMD_4P-L4.2-W3.2-P2.20-LS4.6
- U13: footprint LTC3894EFE:SOP65P640X120-17N -> LTC3894EFE:TSSOP-20_L6.5-W4.4-P0.65-BL-EP
- U14: footprint AP3P3:AP3P3R0MT -> AP3P3R0MT:AP3P3R0MT
- moved J5 274.4 mm to (213.4, 56.3), turned to 90 degrees
- moved U16 268.0 mm to (203.5, 57.4)
- moved R12 260.8 mm to (204.6, 55.0), turned to 180 degrees
- moved R8 260.1 mm to (204.7, 59.8)
- moved C6 227.1 mm to (174.0, 82.1), turned to 180 degrees
- moved C7 219.6 mm to (166.3, 62.9)
- moved TP8 205.5 mm to (146.8, 69.7)
- moved R17 194.6 mm to (130.5, 72.8), turned to 90 degrees
- moved C27 194.4 mm to (129.0, 72.8), turned to -90 degrees
- moved C51 193.5 mm to (130.7, 68.4), turned to -90 degrees
- moved C48 190.5 mm to (125.3, 73.6), turned to 180 degrees
- moved R29 190.5 mm to (129.7, 75.2)
- moved C52 189.1 mm to (138.0, 82.2), turned to -90 degrees
- moved R27 186.4 mm to (125.3, 75.2)
- moved C49 186.0 mm to (120.8, 76.0)
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Connections:
- COM-TO-STM1 pad 3: USART3_RX_STM -> USART3_TX_STM
- COM-TO-STM1 pad 6: USART3_RX_STM -> USART3_TX_STM
- FB1 pad 1: 3V3 -> 3.3VA
- J17 pad 3: USART3_TX_STM -> USART3_RX_STM
- J8 pad 1: VSS -> ROTARY_DC_OUT
- J8 pad 3: ROTARY_DC_OUT -> VSS
- R18 pad 1: SPI1_RESET -> 3V3
- R18 pad 2: RESET1 -> Net-(R18-Pad2)
- R20 pad 1: Net-(SW3-3) -> Net-(R20-Pad1)
- R3 pad 1: Net-(SW1-A) -> Net-(R3-Pad1)
- R48 pad 1: ADC2_INP12 -> ADC1_INP12
- U1 pad 24: USART3_RX_BLE -> USART3_RX_STM
- U1 pad 29: USART3_TX_BLE -> USART3_TX_STM
- U12 pad 1: Net-(U13-RUN) -> IN-24V
- U12 pad 2: Net-(U13-RUN) -> IN-24V
- U12 pad 3: IN-24V -> Net-(U13-RUN)
- U12 pad 4: IN-24V -> Net-(U13-RUN)
- U3 pad 18: SPI1_CLK -> SPI1_SCK
- U5 pad 18: SPI1_CLK -> SPI1_SCK
- U5 pad 4: RESET1 -> RESET
- U6 pad 11: USART3_TX_STM -> USART3_RX_STM
- U6 pad 13: unconnected-(U6-PA0-Pad13) -> Net-(U6-PA0)
- U6 pad 42: unconnected-(U6-PB10-Pad42) -> Net-(U6-PB10)
- U6 pad 8: unconnected-(U6-PA12-Pad8) -> Net-(U6-PA12)
Routing:
- net VSS: track 0.00 -> 1269.3 mm, vias 0 -> 32
- net 5V: track 0.00 -> 528.3 mm, vias 0 -> 12
- net 3V3: track 0.00 -> 333.5 mm, vias 0 -> 13
- net IN-24V: track 0.00 -> 280.9 mm, vias 0 -> 84
- net TIM3_CH4: track 0.00 -> 142.1 mm, vias 0 -> 4
- net UART5_RX_SC: track 0.00 -> 140.2 mm, vias 0 -> 1
- net UART5_TX_SC: track 0.00 -> 136.2 mm, vias 0 -> 1
- net TIM8_CH3: track 0.00 -> 124.9 mm, vias 0 -> 2
- net TIM3_CH2: track 0.00 -> 114.5 mm, vias 0 -> 2
- net SPI1_MOSI: track 0.00 -> 106.2 mm, vias 0 -> 2
- net Rotary_GPIO_Read: track 0.00 -> 102.5 mm, vias 0 -> 2
- net SPI1_SCK: track 0.00 -> 101.5 mm, vias 0 -> 3
- net SPI1_RESET: track 0.00 -> 97.2 mm, vias 0 -> 2
- net SPI1_MISO: track 0.00 -> 91.1 mm, vias 0 -> 4
- net GNDREF: track 0.00 -> 90.7 mm, vias 0 -> 3
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- added copper zone on B.Cu, net IN-24V
- added copper zone on F.Cu, net IN-24V
- added copper zone on B.Cu, net MOTOR_A
- added copper zone on F.Cu, net MOTOR_A
- added copper zone on B.Cu, net MOTOR_B
- added copper zone on F.Cu, net MOTOR_B
- added copper zone on B.Cu, net Net-(D7-A)
- added copper zone on F.Cu, net Net-(D7-A)
- added copper zone on F.Cu, net Net-(D7-K)
- added copper zone on F.Cu, net Net-(D8-K)
- added copper zone on F.Cu, net Net-(U13-RUN)
- added copper zone on B.Cu, net ROTARY_DC_OUT
- added copper zone on F.Cu, net ROTARY_DC_OUT
- added copper zone on B.Cu, net VSS
- added copper zone on F.Cu, net VSS
Other:
- outline, holes or cut-outs redrawn
- copper layers 2 -> 4
- board text added: "24V"
- board text added: "3V3"
- board text added: "5V"
- board text added: "BOOT"
- board text added: "FOOTLOCK"
- board text added: "GND"
- board text added: "INCLINO 1"
- board text added: "INCLINO 2"
- board text added: "IR ROTARY"
- board text added: "LIDAR"
- board text added: "MOTOR A"
- board text added: "MOTOR B"
- board text added: "OUT 1"
- board text added: "OUT 2"
- board text added: "PA0"
- board text added: "PA12"
- board text added: "PB10"
- board text added: "PC0"
- board text added: "PC13"
- board text added: "PD2"
- board text added: "PROG"
- board text added: "PSU"
- board text added: "REMOTE"
- board text added: "RESET"
- board text added: "ROTARY OUT"
- board text added: "RXD"
- board text added: "SC"
- board text added: "SELENOID 1"
- board text added: "SELENOID 2"
- board text added: "SPI1_MOSI"
- board text added: "SPI2_CLK"
- board text added: "SPI2_CS"
- board text added: "SPI2_MOSI"
- board text added: "ST-LINK V3"
- board text added: "STM32H533RET6"
- board text added: "TXD"
- board text added: "USB CDC"
- board text added: "VBAT"
- board text removed: "GYRO 3"
