File: OTMAKSTM32H05_64PIN/OTMAK.kicad_sch (KiCad schematic)
At the start: 82 parts, among them J1 TYPE-C-31-M-12, J10 TX_DEBUG, J11 Conn_01x01, J12 Conn_01x08, J13 Conn_01x08, J15 Conn_01x08, J16 Conn_01x08, J2 TYPE-C-31-M-12, J3 TYPE-C-31-M-12, J4 TYPE-C-31-M-12, J5 TYPE-C-31-M-12, J6 RJ45, J7 STLink, J8 RJ45, J9 RX_DEBUG, Q5 BSS138, SW2 EN, U2 W25Q128JVSIQ, Y1 25.00Mhz, 50PPM, Y2 32.768 kHz

Commit message: update skematik 241205_451
Parts:
- removed J5: TYPE-C-31-M-12, TYPE-C-31-M-12:HRO_TYPE-C-31-M-12, symbol TYPE-C-31-M-12:TYPE-C-31-M-12
- removed R14: 5k1, Resistor_SMD:R_0402_1005Metric, symbol Device:R
- added C85, C86: 2.2uF, Capacitor_SMD:C_0402_1005Metric, symbol Device:C
- added C87: 100nF, Capacitor_SMD:C_0402_1005Metric, symbol Device:C
- added D2: D, symbol Device:D
- added R8: 5k1, Resistor_SMD:R_0402_1005Metric, symbol Device:R
- added U16: USBLC6-2SC6, Package_TO_SOT_SMD:SOT-23-6, symbol Power_Protection:USBLC6-2SC6
- C22: value 22uF -> 100nF; footprint Capacitor_SMD:C_0805_2012Metric -> Capacitor_SMD:C_0402_1005Metric; JLCPCB Part (none) -> C28233
- J4: footprint TYPE-C-31-M-12:HRO_TYPE-C-31-M-12 -> HRO_TYPE-C-31-M-12; JLCPCB Part C165948 -> (none); MANUFACTURER (none) -> HRO Electronics; PARTREV (none) -> A
Connections:
- net I2C_SCL is gone; now on net I2C1_SCL: J1.A7 (DN1), J1.B7 (DN2)
- net I2C_SDA is gone; now on net I2C1_SDA: J1.A6 (DP1), J1.B6 (DP2)
- net LED1 is gone; now on net LD1: R8.1
- net PB3 is gone; now on net Rotary_GPIO_Read: U1.55 (PB3(JTDO/TRACESWO))
- net PB9 is gone; now on net PA15: TP2.1
- net PC12 is gone; now on net LD1: U1.53 (PC12)
- net RESETPIN is gone; now on net SPI1_RESET: R15.1, R18.1
- net SPI3_CLK is gone; now on net SPI2_CLK: TP4.1, U2.6 (SCK)
- net SPI3_CS is gone; now on net SPI2_CS: TP3.1, U2.1 (~{CS})
- net SPI3_MISO is gone; now on net SPI2_MISO: TP6.1, U2.2 (DO(IO1))
- net SPI3_MOSI is gone; now on net SPI2_MOSI: TP5.1, U2.5 (DI(IO0))
- net TIM2_CH2 is gone; now on net TIM2_CH2_BUZZER: U1.15 (PA1)
- net UART4_RX is gone; now on net UART4_RX_LIDAR: J2.A6 (DP1), J2.B7 (DN2)
- net UART4_TX is gone; now on net UART4_TX_LIDAR: J2.A7 (DN1), J2.B6 (DP2)
- net USART1_RX is gone; now on net USART1_RX_ST-LINK: J7.13 (Pin_13)
- net USART1_TX is gone; now on net USART1_TX_ST-LINK: J7.14 (Pin_14)
- net USART3_RX_STM is gone; now on net USART3_RX_BLE: J9.1 (Pin_1)
- net USART3_TX_STM is gone; now on net USART3_TX_BLE: J10.1 (Pin_1)
- net 3V3: no longer U1.13 (VDD)
- net 5V: now also D2.1 (K), U16.5 (VBUS); no longer C22.1
- net GND: now also C22.1, R12.2, C85.1, C86.1, C87.1, R8.1, U16.2 (GND); no longer C22.2, R12.1, U1.12 (VSS)
- net LD1: no longer U1.2 (PC13)
- net SWCLK: now also U1.49 (PA14(SWCLK))
- net SWDIO: no longer U1.49 (PA14(SWCLK))
- net USB-DM: now also U16.3 (I/O2)
- net USB-DP: now also U16.1 (I/O2)
- net VCAP: no longer U1.30 (VCAP)
- net VDDA: now also U1.13 (VDDA)
- net VSSA: now also U1.12 (VSSA)
- net at J4.A4B9 (VBUS), J4.B4A9 (VBUS): now also D2.2 (A)
- net at J4.A5 (CC1): now also R8.2
- net at J4.B5 (CC2): now also R12.1
- net C_D+: now reaches J4.B8 (SBU2)
- net C_D+: now also J4.A6 (DP1), U16.6 (I/O1)
- net BUZZER renamed TIM2_CH2_BUZZER
- net INPUT_Foot_LOCK renamed C_D-
- net C_D-: now also U16.4 (I/O1); no longer J4.A6 (DP1), J4.B6 (DP2)
- net SPI2_SCK renamed SPI2_CLK
- new net PC13: U1.2 (PC13)
- new net VCAP1: C86.2, C87.2, U1.30 (VCAP)
- new net VCAP2: C22.2, C85.2
- no-connect marks 10 -> 9
Other:
- note removed: "FOOTLOCK"
- note removed: "LPUART1"
- moved on the sheet: C13, C6, C7, J1, J10, J2, J3, J6, J8, J9, R1, R10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

Commit message: revision skematik
Parts:
- removed C22, C87: 100nF, Capacitor_SMD:C_0402_1005Metric, symbol Device:C
- removed C3: 1uF, Capacitor_SMD:C_0402_1005Metric, symbol Device:C
- removed C3: 10nF, Capacitor_SMD:C_0402_1005Metric, symbol Device:C
- removed FB2: 600 @ 100mhz, Inductor_SMD:L_0603_1608Metric, symbol Device:FerriteBead
- added J4: TYPE-C-31-M-12, TYPE-C-31-M-12:HRO_TYPE-C-31-M-12, symbol TYPE-C-31-M-12:TYPE-C-31-M-12
- added TP8: ~, TestPoint:TestPoint_Loop_D2.50mm_Drill1.0mm, symbol Connector:TestPoint
- C12: value 10uF -> 1uF
- C13: renamed from C14; value 10uF -> 1uF
- C14: renamed from C15; value 10uF -> 1uF
- C15: renamed from C16; value 10uF -> 1uF
- C2: value 6.8pF -> 24pF
- Y1: value 25.00Mhz, 50PPM -> 24MHz, 6pF
- renumbered C21 to C18, C17 to C19, C25 to C20, C27 to C21, C26 to C22, C24 to C23, C13 to C24, C6 to C25, C7 to C26, C86 to C6, C85 to C7, J4 to J5, J8 to Remote1, J6 to SC1
Connections:
- net SPI1_NSS is gone; now on net SPI1_CS1: U3.17 (CE)
- net SPI2_NSS is gone; now on net SPI1_CS2: U5.17 (CE)
- net VCAP is gone; now on net VCAP2: U1.62 (VCAP2)
- net VREF+ is gone; now on net VDDA: C3.2, C3.2, FB1.2
- net ADC2_INP12: no longer U1.10 (PC2)
- net C_D+: now also J5.B6 (DP2); no longer J5.B8 (SBU2)
- net GND: now also J4.A1B12 (GND), J4.B1A12 (GND), J4.S1 (SHIELD), J4.S2 (SHIELD), J4.S3 (SHIELD), J4.S4 (SHIELD)
- net Rotary_GPIO_Read: no longer U1.60 (BOOT0)
- net USART3_RX_BLE: no longer J9.1 (Pin_1)
- net USART3_TX_BLE: no longer J10.1 (Pin_1)
- net ADC1_INP10 renamed PC0
- net PC0: now also TP8.1
- net LD2 renamed PD2
- net PD2: now also TP2.1
- net PA15 renamed INPUT_Foot_LOCK
- net INPUT_Foot_LOCK: now also J4.A6 (DP1), J4.A7 (DN1), J4.B6 (DP2), J4.B7 (DN2); no longer TP2.1
- new net: J4.A4B9 (VBUS), J4.B4A9 (VBUS)
- new net ADC1_INP12: U1.10 (PC2)
- new net BOOT: U1.60 (BOOT0)
- new net USART3_RX_STM: J9.1 (Pin_1)
- new net USART3_TX_STM: J10.1 (Pin_1)
Other:
- sheet BLE_MOBILE ports: added UART_RXD_BLE, UART_TXD_BLE; removed UART_RXD_STM, UART_TXD_STM
- sheet PowerDriver ports: added ADC1_INP0, ADC2_INP11, ADC2_INP12, ADC2_INP13, TIM3_CH1, TIM3_CH2, TIM3_CH3, TM3_CH4, TM8_CH3, TM8_CH4; removed ADC1IN, ADC_OUT1, ADC_OUT2, ADC_OUT3, ADC_OUT4, IN1, IN3, IN4, TM1_CH1, TM1_CH3, TM1_CH4
- note added: "FOOTLOCK"
- note added: "USB CDC"
- moved on the sheet: C3, C6, C7, FB1, L1, Remote1, SC1, U16

Commit message: next revisi 241206 1656
Parts:
- D2: JLCPCB Part (none) -> C81598
- J5: JLCPCB Part (none) -> C165948
Connections:
- net USART3_RX_BLE is gone; now on net USART3_RX_STM: U1.24 (PC4)
- net USART3_TX_BLE is gone; now on net USART3_TX_STM: U1.29 (PB10)
Other:
- sheet BLE_MOBILE ports: added UART_RXD_STM, UART_TXD_STM; removed UART_RXD_BLE, UART_TXD_BLE
- note added: "RX_BLE(PA8)"
- note added: "TX_BLE(PA9)"
- moved on the sheet: L1
Changed lines of the file:
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@@
 	)
 	(junction
+		(at 327.66 81.28)
+		(diameter 0)
+		(color 0 0 0 0)
+	)
+	(junction
 		(at 151.13 262.89)
 		(diameter 0)
@@
 	)
 	(junction
+		(at 331.47 81.28)
+		(diameter 0)
+		(color 0 0 0 0)
+	)
+	(junction
 		(at 293.37 156.21)
 		(diameter 0)
@@
 	(wire
 		(pts
+			(xy 331.47 81.28) (xy 350.52 81.28)
+		)
+		(stroke
+			(width 0)
+			(type default)
+		)
+	)
+	(wire
+		(pts
 			(xy 132.08 30.48) (xy 123.19 30.48)
 		)
@@
 	(wire
 		(pts
+			(xy 327.66 81.28) (xy 327.66 83.82)
+		)
+		(stroke
+			(width 0)
+			(type default)
+		)
+	)
+	(wire
+		(pts
 			(xy 73.66 260.35) (xy 74.93 260.35)
 		)
@@
 	(wire
 		(pts
+			(xy 327.66 81.28) (xy 308.61 81.28)
+		)
+		(stroke
+			(width 0)
+			(type default)
+		)
+	)
+	(wire
+		(pts
 			(xy 364.49 236.22) (xy 364.49 238.76)
 		)
@@
 	(wire
 		(pts
+			(xy 308.61 67.31) (xy 308.61 81.28)
+		)
+		(stroke
+			(width 0)
+			(type default)
+		)
+	)
+	(wire
+		(pts
 			(xy 153.67 140.97) (xy 163.83 140.97)
 		)
@@
 	(wire
 		(pts
-			(xy 327.66 80.01) (xy 327.66 83.82)
+			(xy 327.66 80.01) (xy 327.66 81.28)
 		)
 		(stroke
@@
 	(wire
 		(pts
+			(xy 331.47 81.28) (xy 331.47 83.82)
+		)
+		(stroke
+			(width 0)
+			(type default)
+		)
+	)
+	(wire
+		(pts
 			(xy 217.17 212.09) (xy 217.17 217.17)
 		)
@@
 	(wire
 		(pts
+			(xy 350.52 67.31) (xy 350.52 81.28)
+		)
+		(stroke
+			(width 0)
+			(type default)
+		)
+	)
+	(wire
+		(pts
 			(xy 63.5 60.96) (xy 63.5 64.77)
 		)
@@
 	(wire
 		(pts
-			(xy 331.47 80.01) (xy 331.47 83.82)
+			(xy 331.47 80.01) (xy 331.47 81.28)
 		)
 		(stroke
@@
 	(wire
 		(pts
-			(xy 213.36 49.53) (xy 224.79 49.53)
+			(xy 213.36 49.53) (xy 218.44 49.53)
 		)
 		(stroke
@@
 		)
 	)
+	(wire
+		(pts
+			(xy 226.06 49.53) (xy 227.33 49.53)
+		)
+		(stroke
+			(width 0)
+			(type default)
+		)
+	)
 	(text "DEBUG LED"
 		(exclude_from_sim no)
@@
 		)
 	)
+	(text "RX_BLE(PA8)\n"
+		(exclude_from_sim no)
+		(at 350.774 66.04 0)
+		(effects
+			(font
+				(size 1.27 1.27)
+			)
+		)
+	)
 	(text "Control Unit"
 		(exclude_from_sim no)
@@
 		)
 	)
+	(text "TX_BLE(PA9)\n"
+		(exclude_from_sim no)
+		(at 307.594 66.04 0)
+		(effects
+			(font
+				(size 1.27 1.27)
+			)
+		)
+	)
 	(text "TERMINAL BLOK"
 		(exclude_from_sim no)
@@
 		)
 	)
-	(global_label "USART3_RX_BLE"
+	(global_label "USART3_RX_STM"
 		(shape input)
 		(at 95.25 113.03 270)
@@
 		)
 		(property "Intersheetrefs" "${INTERSHEET_REFS}"
-			(at 95.25 130.9527 90)
+			(at 95.25 131.1341 90)
 			(effects
 				(font
@@
 		)
 	)
-	(global_label "USART3_TX_BLE"
+	(global_label "USART3_TX_STM"
 		(shape input)
 		(at 107.95 113.03 270)
@@
 		)
 		(property "Intersheetrefs" "${INTERSHEET_REFS}"
-			(at 107.95 130.6503 90)
+			(at 107.95 130.8317 90)
 			(effects
 				(font
@@
 			)
 		)
+		(property "JLCPCB Part" "C165948"
+			(at 212.09 191.77 0)
+			(effects
+				(font
+					(size 1.27 1.27)
+				)
+				(hide yes)
+			)
+		)
 		(pin "A4B9"
 		)
@@
 		(lib_name "GNDREF_1")
 		(lib_id "power:GNDREF")
-		(at 232.41 49.53 0)
+		(at 227.33 49.53 0)
 		(mirror y)
 		(unit 1)
@@
 		(dnp no)
 		(property "Reference" "#PWR011"
-			(at 232.41 55.88 0)
+			(at 227.33 55.88 0)
 			(effects
 				(font
@@
 		)
 		(property "Value" "GND"
-			(at 232.41 53.975 0)
+			(at 227.33 53.975 0)
 			(effects
 				(font
@@
 		)
 		(property "Footprint" ""
-			(at 232.41 49.53 0)
+			(at 227.33 49.53 0)
 			(effects
 				(font
@@
 		)
 		(property "Datasheet" ""
-			(at 232.41 49.53 0)
+			(at 227.33 49.53 0)
 			(effects
 				(font
@@
 		)
 		(property "Description" ""
-			(at 232.41 49.53 0)
+			(at 227.33 49.53 0)
 			(effects
 				(font
@@
 			)
 		)
+		(property "JLCPCB Part" "C81598"
+			(at 236.22 181.61 0)
+			(effects
+				(font
+					(size 1.27 1.27)
+				)
+				(hide yes)
+			)
+		)
 		(pin "2"
 		)
@@
 	(symbol
 		(lib_id "Device:L")
-		(at 228.6 49.53 90)
+		(at 222.25 49.53 90)
 		(unit 1)
 		(exclude_from_sim no)
@@
 		(fields_autoplaced yes)
 		(property "Reference" "L1"
-			(at 228.6 44.45 90)
+			(at 222.25 44.45 90)
 			(effects
 				(font
@@
 		)
 		(property "Value" "L"
-			(at 228.6 46.99 90)
+			(at 222.25 46.99 90)
 			(effects
 				(font
@@
 		)
 		(property "Footprint" "Inductor_SMD:L_0402_1005Metric"
-			(at 228.6 49.53 0)
+			(at 222.25 49.53 0)
 			(effects
 				(font
@@
 		)
 		(property "Datasheet" "~"
-			(at 228.6 49.53 0)
+			(at 222.25 49.53 0)
 			(effects
 				(font
@@
 		)
 		(property "Description" "Inductor"
-			(at 228.6 49.53 0)
+			(at 222.25 49.53 0)
 			(effects
 				(font
@@
 			)
 		)
-		(pin "UART_TXD_BLE" input
+		(pin "UART_RXD_STM" input
 			(at 327.66 83.82 90)
 			(effects
@@
 			)
 		)
-		(pin "UART_RXD_BLE" input
+		(pin "UART_TXD_STM" input
 			(at 331.47 83.82 90)
 			(effects

Commit message: full version
Parts:
- removed C21: 0.1uF, Capacitor_SMD:C_0805_2012Metric, symbol Device:C
- removed R18: 100R, Resistor_SMD:R_0402_1005Metric, symbol Device:R
- added C58: 100nF, Capacitor_SMD:C_0402_1005Metric, symbol Device:C
- added C60: 22uF, Capacitor_SMD:C_0805_2012Metric, symbol Device:C
- added J14: TYPE-C-31-M-12, USB_Type_C:HRO_TYPE-C-31-M-12, symbol TYPE-C-31-M-12:TYPE-C-31-M-12
- added R35, R38: 5k1, Resistor_SMD:R_0402_1005Metric, symbol Device:R
- added TP10: ~, TestPoint:TestPoint_Loop_D2.50mm_Drill1.0mm, symbol Connector:TestPoint
- D2: footprint (none) -> Diode_SMD:D_SOD-123
- J1, J2, J3, J4: footprint TYPE-C-31-M-12:HRO_TYPE-C-31-M-12 -> USB_Type_C:HRO_TYPE-C-31-M-12
- J12, J13, J15, J16: footprint Terminal_8_pin:TerminalBlock_8_pin -> TerminalBlock_8_pin:TerminalBlock_8_pin
- J5: footprint HRO_TYPE-C-31-M-12 -> USB_Type_C:HRO_TYPE-C-31-M-12
- SW2: footprint TS-1187A-B-A-B:SW_TS-1187A-B-A-B -> Push Button:KEY-SMD_4P-L4.2-W3.2-P2.20-LS4.6
Connections:
- net RESET1 is gone; now on net RESET: U5.4 (RESET)
- net SPI1_CLK is gone; now on net SPI1_SCK: U3.18 (SCLK), U5.18 (SCLK)
- net 3V3: no longer FB1.1
- net 5V: now also C60.1, J14.A4B9 (VBUS), J14.B4A9 (VBUS)
- net GND: now also C58.2, C60.2, J14.A1B12 (GND), J14.B1A12 (GND), J14.S1 (SHIELD), J14.S2 (SHIELD), J14.S3 (SHIELD), J14.S4 (SHIELD), R35.1, R38.2
- net NRST: now also SW2.1, SW2.2; no longer SW2.A, SW2.B (2)
- net PC13: now also TP10.1
- net USART2_RX_PSU: now also J14.A7 (DN1), J14.B7 (DN2)
- net USART2_TX_PSU: now also J14.A6 (DP1), J14.B6 (DP2)
- net at TP1.1, U1.1 (VBAT): now also C58.1
- new net: J14.A5 (CC1), R35.2
- new net: J14.B5 (CC2), R38.1
- new net: R3.1, SW2.3, SW2.4
- new net 3.3VA: FB1.1
Other:
- sheet PowerDriver ports: added ADC1_INP12; removed ADC2_INP12
- moved on the sheet: C24, C25, C26, J1, J2, J3, J4, R1, R10, R2, R5, R7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
