File: OTMAKSTM32H05_64PIN/PowerDriver.kicad_sch (KiCad schematic)
At the start: 99 parts, among them J18 IR Interrupt, J19 Conn_01x08, J20 MOTOR_A/MOTOR_B, J21 24V INPUT, U11 LM393, U12 CC6900SO-20A, U15 LM1117-3.3

Commit message: update skematik 241205_451
Other:
- moved on the sheet: C1, C10, C11, C12, C13, C2, C3, C4, C56, C65, R1, R2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

Commit message: revision skematik
Parts:
- removed C52, C81, C84: 100nF, Capacitor_SMD:C_0805_2012Metric, symbol Device:C
- removed C54, C55: 10nF, Capacitor_SMD:C_0603_1608Metric, symbol Device:C
- removed C57, C58: 100nF, Capacitor_SMD:C_1206_3216Metric, symbol Device:C
- removed C60, C61: 470uF/1000uF, Capacitor_SMD:CP_Elec_10x10.5, symbol Device:C_Polarized
- removed C79, C82: 1uF, Capacitor_SMD:C_0805_2012Metric, symbol Device:C
- removed J19: Conn_01x08, Terminal_8_pin:TerminalBlock_8_pin, symbol Connector_Generic:Conn_01x08
- removed J20: MOTOR_A/MOTOR_B, Terminal_4_pin:TerminalBlock_4_pin, symbol Connector_Generic:Conn_01x04
- removed R33: 10K, Capacitor_SMD:C_0603_1608Metric, symbol Device:R
- removed R34: 0.51K, Resistor_SMD:R_0603_1608Metric, symbol Device:R
- removed R35: 0.51K, Resistor_SMD:R_0805_2012Metric, symbol Device:R
- removed R38, R39: 10K, Resistor_SMD:R_0603_1608Metric, symbol Device:R
- removed R41, R43: 47K, Resistor_SMD:R_0603_1608Metric, symbol Device:R
- removed R42, R44: 0R, Resistor_SMD:R_0805_2012Metric, symbol Device:R
- removed U15: LM1117-3.3, Package_TO_SOT_SMD:SOT-223-3_TabPin2, symbol Regulator_Linear:LM1117-3.3
- removed U8: ~, Package_TO_SOT_SMD:TO-263-7_TabPin8, symbol IFX007T:IFX007T
- added C27: 1nF, Capacitor_SMD:C_0603_1608Metric, symbol Device:C
- added C52: 470uF/1000uF, Capacitor_SMD:CP_Elec_10x10.5, symbol Device:C_Polarized
- added C88: 4.7nF, Capacitor_SMD:C_0805_2012Metric, symbol Device:C
- added J6: MOTOR_A/MOTOR_B, symbol Connector_Generic:Conn_01x06
- added J8: ROTARY, symbol Connector_Generic:Conn_01x03
- added R14: 30.1K, Resistor_SMD:R_0603_1608Metric, symbol Device:R
- added R17: 1K, Resistor_SMD:R_0603_1608Metric, symbol Device:R
- added R19: 10K, Capacitor_SMD:C_0603_1608Metric, symbol Device:R
- added R6: 52.3K, Resistor_SMD:R_0603_1608Metric, symbol Device:R
- added U4: TPS73601DBVR, easyeda2kicad:SOT-23-5_L3.0-W1.7-P0.95-LS2.8-BR, symbol TPS73601DBVR:TPS73601DBVR
- C48: value 1nF -> 100nF
- C49: value 1nF -> 1uF; footprint Capacitor_SMD:C_0805_2012Metric -> Capacitor_SMD:C_0603_1608Metric; JLCPCB Part (none) -> C28323
- C51: footprint Capacitor_SMD:C_0603_1608Metric -> Capacitor_SMD:C_1206_3216Metric
- C56, C65: value 10nF -> 1uF
- C75: value 22uF -> 4.7uF
- C76: value 10uF -> 4.7nF
- R26: value 1K -> 10K; footprint Resistor_SMD:R_0603_1608Metric -> Capacitor_SMD:C_0603_1608Metric
- R27: value 1K -> 0.51K; footprint Resistor_SMD:R_0805_2012Metric -> Resistor_SMD:R_0603_1608Metric
- R29: value 10K -> 3.9K; footprint Capacitor_SMD:C_0603_1608Metric -> Resistor_SMD:R_0603_1608Metric
- R30: value 10K -> 33K; footprint Capacitor_SMD:C_0603_1608Metric -> Resistor_SMD:R_0603_1608Metric
- R32: value 10K -> 0R; footprint Capacitor_SMD:C_0603_1608Metric -> Resistor_SMD:R_0805_2012Metric
- R40, R49: value 10K -> 3.9K
- R45, R47: value 47K -> 33K
Connections:
- net 3V3: now also C76.1, C88.1, R6.1, U4.5 (OUT)
- net 5V: now also U4.1 (IN), U4.3 (EN); no longer C76.1
- net GND: now also C56.2, C65.2, R29.2, R40.2, R49.2, C27.2, C52.2, C88.2, J6.1 (Pin_1), J6.2 (Pin_2), J8.1 (Pin_1), R14.2, R17.1, U4.2 (GND); no longer C76.2, R26.1
- net IN-24V: now also C51.1, C52.1
- net MOTOR_A: now also J6.3 (Pin_3), J6.4 (Pin_4)
- net MOTOR_B: now also J6.5 (Pin_5), J6.6 (Pin_6)
- net ROTARY_DC_OUT: now also R30.1, J8.2 (Pin_2), J8.3 (Pin_3)
- net at R30.2: now also C49.1, R29.1, R32.2
- net at R27.2: now also C48.1, U7.5 (SR); no longer C49.1
- net at U7.2 (IN): now also R19.2; no longer R29.2
- net at U7.3 (INH): now also R26.2; no longer R32.2
- net ADC1IN renamed ADC1_INP0
- net ADC_OUT1 renamed ADC2_INP12
- net ADC_OUT2 renamed ADC2_INP11
- net IN1 renamed TIM3_CH1
- net IN3 renamed TIM3_CH2
- removed net IN4: R29.1, R30.1
- net TM1_CH1 renamed TM8_CH3
- net TM1_CH3 renamed TM3_CH4
- net TM1_CH4 renamed ADC2_INP13
- new net: C27.1, R17.2, U7.6 (IS)
- new net: C76.2, R14.1, R6.2, U4.4 (NR/FB)
- new net TIM3_CH3: R19.1
- new net TM8_CH4: R26.1
Other:
- note removed: "JUMPER"
- note removed: "MOTOR PUMP"
- note removed: "MOTOR ROTARY"
- note removed: "SOLENOID PUMP"
- moved on the sheet: D10, D9, R63

Commit message: next revisi 241206 1656
Parts:
- J6: footprint (none) -> TerminalBlock:TerminalBlock_bornier-6_P5.08mm
- J8: footprint (none) -> TerminalBlock:TerminalBlock_bornier-3_P5.08mm
Changed lines of the file:
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@@
 			)
 		)
-		(property "Footprint" ""
+		(property "Footprint" "TerminalBlock:TerminalBlock_bornier-3_P5.08mm"
 			(at 63.5 232.41 0)
 			(effects
@@
 			)
 		)
-		(property "Footprint" ""
+		(property "Footprint" "TerminalBlock:TerminalBlock_bornier-6_P5.08mm"
 			(at 91.44 232.41 0)
 			(effects

Commit message: full version
Parts:
- removed D9: BZV55B5V1, Diode_SMD:D_MiniMELF, symbol Device:D_Zener
- removed J6: MOTOR_A/MOTOR_B, TerminalBlock:TerminalBlock_bornier-6_P5.08mm, symbol Connector_Generic:Conn_01x06
- added C54: 4.7uF, Capacitor_SMD:C_0805_2012Metric, symbol Device:C
- added C55, C57: 4.7nF, Capacitor_SMD:C_0805_2012Metric, symbol Device:C
- added J19, J20, J22: Conn_01x02, TerminalBlock_2_pin:TerminalBlock_2_Pin, symbol Connector_Generic:Conn_01x02
- added R33: 52.3K, Resistor_SMD:R_0603_1608Metric, symbol Device:R
- added R34: 30.1K, Resistor_SMD:R_0603_1608Metric, symbol Device:R
- added TP11, TP12, TP9: ~, TestPoint:TestPoint_Loop_D2.50mm_Drill1.0mm, symbol Connector:TestPoint
- added U8: TPS73601DBVR, Package_TO_SOT_SMD:TSOT-23-5, symbol TPS73601DBVR:TPS73601DBVR
- added ZD1: BZX55C5V1, BZX55C5V1:DO-35_BD2.0-L4.0-P8.00-D0.5-FD, symbol BZX55C5V1:BZX55C5V1_C34365
- C12, C13: footprint Capacitor_SMD:C_0805_2012Metric -> Capacitor_SMD:C_0603_1608Metric
- D8: footprint PDS4150:PDS4150 -> PDS4150-13:POWERDI-5_L5.4-W4.0-LS6.5-RD
- F1: footprint FuseSA72SB0:RES-SMD_SA72SB0 -> fuseSA72SB0:RES-SMD_SA72SB0
- J8: footprint TerminalBlock:TerminalBlock_bornier-3_P5.08mm -> TerminalBlock_3_pin:TerminalBlock_3_Pin
- R8: footprint Resistor_SMD:R_0805_2012Metric -> Resistor_SMD:R_0603_1608Metric
- U14: footprint AP3P3:AP3P3R0MT -> AP3P3R0MT:AP3P3R0MT
- U4: footprint easyeda2kicad:SOT-23-5_L3.0-W1.7-P0.95-LS2.8-BR -> Package_TO_SOT_SMD:TSOT-23-5
Connections:
- net 5V: now also C54.1, TP11.1, TP12.1, TP9.1, U8.1 (IN), U8.3 (EN), ZD1.2 (K)
- net GND: now also J8.3 (Pin_3), C54.2, C57.2, J22.1 (Pin_1), J22.2 (Pin_2), R34.2, U8.2 (GND), ZD1.1 (A); no longer J8.1 (Pin_1)
- net IN-24V: now also U12.1 (IP+), U12.2 (IP+); no longer U12.3 (IP-), U12.4 (IP-)
- net MOTOR_A: now also J19.1 (Pin_1), J19.2 (Pin_2)
- net MOTOR_B: now also J20.1 (Pin_1), J20.2 (Pin_2)
- net ROTARY_DC_OUT: now also J8.1 (Pin_1); no longer J8.3 (Pin_3)
- net at C72.1, C74.1, F1.2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: now also U12.3 (IP-), U12.4 (IP-); no longer U12.1 (IP+), U12.2 (IP+)
- net ADC2_INP12 renamed ADC1_INP12
- new net: C55.2, R33.2, R34.1, U8.4 (NR/FB)
- new net 3.3VA: C55.1, C57.1, R33.1, U8.5 (OUT)
Other:
- moved on the sheet: D10, J8, R63
